File: hdmi-switch-project.sch (KiCad schematic (older format))
At the start: 6 parts, among them J1 HDMI_A_1.4, J2 HDMI_A_1.4, J3 HDMI_A_1.4, J4 HDMI_A_1.4, U1 TMDS442_single_unit

Commit message: Control board has bijuterie now
Signed-off-by: Andrej Manduch <amanduch@gmail.com>
Connections:
- net GND: no longer J1.11 (CKS), J1.2 (D2S), J1.5 (D1S), J1.8 (D0S), J1.SH, J2.11 (CKS), J2.2 (D2S), J2.5 (D1S), J2.8 (D0S), J2.SH, J3.11 (CKS), J3.2 (D2S), J3.5 (D1S), J3.8 (D0S), J3.SH, J4.11 (CKS), J4.2 (D2S), J4.5 (D1S), J4.8 (D0S)
- net SHIELD: now reaches J4.SH
- net SHIELD: now also J1.11 (CKS), J1.2 (D2S), J1.5 (D1S), J1.8 (D0S), J1.SH, J2.11 (CKS), J2.2 (D2S), J2.5 (D1S), J2.8 (D0S), J2.SH, J4.11 (CKS), J4.2 (D2S), J4.5 (D1S), J4.8 (D0S)
- new net SHLIELD: J3.11 (CKS), J3.2 (D2S), J3.5 (D1S), J3.8 (D0S), J3.SH
Other:
- moved on the sheet: J1, J2, J3, J4, R_VSDAJ1, U1

Commit message: Initial devel design
Signed-off-by: Andrej Manduch <amanduch@gmail.com>
Parts:
- removed J1, J2, J3, J4: HDMI_A_1.4, Connector_HDMI:HDMI_A_Contact_Technology_HDMI-19APL2_Horizontal, symbol Connector:HDMI_A_1.4
- removed R_VSDAJ1: 4K6, Resistor_SMD:R_1020_2550Metric, symbol Device:R
- removed U1: TMDS442_single_unit, Package_QFP:TQFP-128_14x14mm_P0.4mm, symbol Interface_HDMI:TMDS442_single_unit
