File: power_input.sch (KiCad schematic (older format))
At the start: 7 parts

Commit message: Initial devel design
Signed-off-by: Andrej Manduch <amanduch@gmail.com>
Parts:
- gave numbers to parts that had none: 6
- renumbered R_ATX_ON to R_ATX_ON1
Changed lines of the file:
@@
 $Descr A4 11693 8268
 encoding utf-8
-Sheet 3 3
+Sheet 2 4
 Title ""
 Date ""
@@
 $EndDescr
 $Comp
-L Connector:ATX-20 J?
+L Connector:ATX-20 J1
 U 1 1 5F7CBCCC
 P 2250 1900
-F 0 "J?" H 2250 2567 50  0000 C CNN
+F 0 "J1" H 2250 2567 50  0000 C CNN
 F 1 "ATX-20" H 2250 2476 50  0000 C CNN
 F 2 "" H 2250 1800 50  0001 C CNN
@@
 $EndComp
 $Comp
-L power:GND #PWR?
+L power:GND #PWR01
 U 1 1 5F7CCFBC
 P 2250 2600
-F 0 "#PWR?" H 2250 2350 50  0001 C CNN
+F 0 "#PWR01" H 2250 2350 50  0001 C CNN
 F 1 "GND" H 2255 2427 50  0000 C CNN
 F 2 "" H 2250 2600 50  0001 C CNN
@@
 $EndComp
 $Comp
-L power:+5V #PWR?
+L power:+5V #PWR02
 U 1 1 5F7CD372
 P 4600 1800
-F 0 "#PWR?" H 4600 1650 50  0001 C CNN
+F 0 "#PWR02" H 4600 1650 50  0001 C CNN
 F 1 "+5V" V 4615 1928 50  0000 L CNN
 F 2 "" H 4600 1800 50  0001 C CNN
@@
 $EndComp
 $Comp
-L power:+3.3V #PWR?
+L power:+3.3V #PWR03
 U 1 1 5F7CDDDA
 P 4600 2000
-F 0 "#PWR?" H 4600 1850 50  0001 C CNN
+F 0 "#PWR03" H 4600 1850 50  0001 C CNN
 F 1 "+3.3V" V 4615 2128 50  0000 L CNN
 F 2 "" H 4600 2000 50  0001 C CNN
@@
 NoConn ~ 2750 2200
 $Comp
-L Switch:SW_DIP_x01 SW?
+L Switch:SW_DIP_x01 SW1
 U 1 1 5F7CEB17
 P 1150 1950
-F 0 "SW?" V 1104 2080 50  0000 L CNN
+F 0 "SW1" V 1104 2080 50  0000 L CNN
 F 1 "SW_DIP_x01" V 1195 2080 50  0000 L CNN
 F 2 "" H 1150 1950 50  0001 C CNN
@@
 	1150 2250 1150 2550
 $Comp
-L Device:R R_ATX_ON
+L Device:R R_ATX_ON1
 U 1 1 5F7D0032
 P 1600 2550
-F 0 "R_ATX_ON" V 1393 2550 50  0000 C CNN
+F 0 "R_ATX_ON1" V 1393 2550 50  0000 C CNN
 F 1 "0R" V 1484 2550 50  0000 C CNN
 F 2 "" V 1530 2550 50  0001 C CNN
@@
 	2250 2550 2250 2600
 $Comp
-L Device:CP C_PWR?
+L Device:CP C_PWR1
 U 1 1 5F7D24ED
 P 3000 2200
-F 0 "C_PWR?" H 3118 2246 50  0000 L CNN
+F 0 "C_PWR1" H 3118 2246 50  0000 L CNN
 F 1 "2200u" H 3118 2155 50  0000 L CNN
 F 2 "" H 3038 2050 50  0001 C CNN
@@
 $EndComp
 $Comp
-L Device:CP C_PWR?
+L Device:CP C_PWR2
 U 1 1 5F7D2C8B
 P 3500 2200
-F 0 "C_PWR?" H 3618 2246 50  0000 L CNN
+F 0 "C_PWR2" H 3618 2246 50  0000 L CNN
 F 1 "2200u" H 3618 2155 50  0000 L CNN
 F 2 "" H 3538 2050 50  0001 C CNN
@@
 $EndComp
 $Comp
-L Device:CP C_PWR?
+L Device:CP C_PWR3
 U 1 1 5F7D313A
 P 4000 2200
-F 0 "C_PWR?" H 4118 2246 50  0000 L CNN
+F 0 "C_PWR3" H 4118 2246 50  0000 L CNN
 F 1 "2200u" H 4118 2155 50  0000 L CNN
 F 2 "" H 4038 2050 50  0001 C CNN
@@
 $EndComp
 $Comp
-L Device:CP C_PWR?
+L Device:CP C_PWR4
 U 1 1 5F7D426E
 P 4500 2200
-F 0 "C_PWR?" H 4618 2246 50  0000 L CNN
+F 0 "C_PWR4" H 4618 2246 50  0000 L CNN
 F 1 "2200u" H 4618 2155 50  0000 L CNN
 F 2 "" H 4538 2050 50  0001 C CNN
