File: stm_control.sch (KiCad schematic (older format))
At the start: 25 parts

Commit message: Initial devel design
Signed-off-by: Andrej Manduch <amanduch@gmail.com>
Parts:
- added C_BUTTON1, C_PWR_CAN1: u1, symbol Device:C
- added D_LED1: LED, symbol Device:LED
- added J_COMM_CAN1, J_COMM_TWI1: Conn_01x02_Male, symbol Connector:Conn_01x02_Male
- added R_BTN1, R_RST1: 10K, symbol Device:R
- added R_CAN_TERM1: 120R, symbol Device:R
- added R_LED1: 510R, symbol Device:R
- added SW_STM1: SW_Push, symbol Switch:SW_Push
- added U2: TCAN330, symbol Interface_CAN_LIN:TCAN330
- gave numbers to parts that had none: 5
- renumbered C_SRV_PROG to C_SRV_PROG1, J_BOOT_JUMPER to J_BOOT_JUMPER1, J_SERVICE_PROG to J_SERVICE_PROG1, J_SERVICE_USB to J_SERVICE_USB1, TP_PROG_CLCK to TP_PROG_CLCK1, TP_PROG_GND to TP_PROG_GND1, TP_PROG_IO to TP_PROG_IO1, XTAL_STM2_RTC to XTAL_STM2_RTC1
Connections:
- net +3V3: now also C_PWR_CAN1.2, D_LED1.2 (A), R_BTN1.1, U2.3 (VCC)
- net GND: now also C_BUTTON1.2, SW_STM1.1
- net STM_GPIO0: now reaches U3.10 (PA0)
- net STM_GPIO1: now reaches U3.11 (PA1)
- net STM_GPIO2: now reaches U3.12 (PA2)
- net STM_GPIO3: now reaches U3.13 (PA3)
- net STM_GPIO4: now reaches U3.14 (PA4)
- net STM_GPIO5: now reaches U3.15 (PA5)
- net STM_GPIO6: now reaches U3.16 (PA6)
- net STM_GPIO7: now reaches U3.17 (PA7)
- net STM_GE: now reaches U3.18 (PB0)
- net STM_GPIO: now reaches U3.19 (PB1)
- net STM_LED1: now reaches U3.2 (PC13)
- net STM_LED1: now also R_LED1.1
- net STM_CNTRL_CLK: now reaches U3.21 (PB10)
- net STM_CNTRL_CLK: now also J_COMM_TWI1.1 (Pin_1)
- net STM_CNTRL_SDA: now reaches U3.22 (PB11)
- net STM_CNTRL_SDA: now also J_COMM_TWI1.2 (Pin_2)
- net STM_BTN1: now reaches U3.28 (PB15)
- net STM_BTN1: now also C_BUTTON1.1, R_BTN1.2, SW_STM1.2
- net STM_GPIO8: now reaches U3.29 (PA8)
- net STM_TX: now reaches U3.30 (PA9)
- net STM_RX: now reaches U3.31 (PA10)
- net STM_GPIO9: now reaches U3.38 (PA15)
- net STM_A0: now reaches U3.39 (PB3)
- net STM_A1: now reaches U3.40 (PB4)
- net STM_OVS: now reaches U3.41 (PB5)
- net ST_H_CLK: now reaches U3.42 (PB6)
- net ST_H_SDA: now reaches U3.43 (PB7)
- net STM_CAN_RX: now reaches U3.45 (PB8)
- net STM_CAN_RX: now also U2.4 (RXD)
- net STM_CAN_TX: now reaches U3.46 (PB9)
- net STM_CAN_TX: now also U2.1 (TXD)
- net at U3.7 (NRST): now also R_RST1.2
- new net: C_PWR_CAN1.1, U2.2 (GND)
- new net: J_COMM_CAN1.2 (Pin_2), R_CAN_TERM1.2, U2.6 (CANL)
- new net: J_COMM_CAN1.1 (Pin_1), R_CAN_TERM1.1, U2.7 (CANH)
- new net: D_LED1.1 (K), R_LED1.2
- new net VCC: R_RST1.1
Other:
- note added: "Communication\n\nTWI & CAN (not necessary for first devel board)"
- note added: "Devel board only"
- note added: "Example Button"
- note added: "Example LED"
- moved on the sheet: C_SRV_PROG1, TP_PROG_GND1, TP_PROG_VCC33

Commit message: shield typo fixed
Signed-off-by: Andrej Manduch <amanduch@gmail.com>
Connections:
- net SHLIELD renamed SHIELD
Changed lines of the file:
@@
 	1150 3150 1150 3100
 Text GLabel 950  3150 0    50   Input ~ 0
-SHLIELD
+SHIELD
 Wire Wire Line
 	950  3150 1050 3150
