File: hdmi-switch-project/HDMI_Connector.sch (KiCad schematic (older format))
At the start: 3 parts

Commit message: Changed shielding for HDMI
For input ports added 0R between shielding so it can be removed

Signed-off-by: Andrej Manduch <amanduch@gmail.com>
Connections:
- net SHIELD renamed SH
Changed lines of the file:
@@
 $Descr A4 11693 8268
 encoding utf-8
-Sheet 9 10
+Sheet 6 10
 Title ""
 Date ""
@@
 Comment4 ""
 $EndDescr
-Text GLabel 5150 4500 0    50   Input ~ 0
-SHIELD
 Wire Wire Line
 	5650 4650 5450 4650
@@
 Wire Wire Line
 	5250 4500 5350 4500
-Wire Wire Line
-	5150 4500 5250 4500
-Connection ~ 5250 4500
 $Comp
 L Connector:HDMI_A_1.4 J?
@@
 	4000 5050 4000 4950
 Connection ~ 4250 5050
+Text HLabel 5850 4500 2    50   Input ~ 0
+SH
+Wire Wire Line
+	5850 4500 5750 4500
+Connection ~ 5750 4500
 $EndSCHEMATC
