File: hdmi-switch-project/hdmi_circuit.sch (KiCad schematic (older format))
At the start: 12 parts, among them U1 TMDS442_single_unit

Commit message: Changed shielding for HDMI
For input ports added 0R between shielding so it can be removed

Signed-off-by: Andrej Manduch <amanduch@gmail.com>
Parts:
- added R? (x4): R0, symbol Device:R
Connections:
- net labels added: SHIELD
- wire segments 280 -> 296
Changed lines of the file:
@@
 	3700 6650 3800 6650
 $Sheet
-S 8700 650  600  1600
+S 8650 650  600  1600
 U 5F55479C
 F0 "sheet5F55478E" 50
 F1 "HDMI_Connector.sch" 50
-F2 "D2+" I L 8700 850 50
-F3 "D2-" I L 8700 950 50
-F4 "D1+" I L 8700 1050 50
-F5 "D1-" I L 8700 1150 50
-F6 "D0+" I L 8700 1250 50
-F7 "D0-" I L 8700 1350 50
-F8 "CK+" I L 8700 1450 50
-F9 "CK-" I L 8700 1550 50
-F10 "SCL" I L 8700 1700 50
-F11 "SDA" I L 8700 1800 50
-F12 "HPD" I L 8700 1950 50
-F13 "HDMI_5V" I L 8700 2100 50
+F2 "D2+" I L 8650 850 50
+F3 "D2-" I L 8650 950 50
+F4 "D1+" I L 8650 1050 50
+F5 "D1-" I L 8650 1150 50
+F6 "D0+" I L 8650 1250 50
+F7 "D0-" I L 8650 1350 50
+F8 "CK+" I L 8650 1450 50
+F9 "CK-" I L 8650 1550 50
+F10 "SCL" I L 8650 1700 50
+F11 "SDA" I L 8650 1800 50
+F12 "HPD" I L 8650 1950 50
+F13 "HDMI_5V" I L 8650 2100 50
+F14 "SH" I R 9250 850 50
 $EndSheet
 Wire Wire Line
@@
 F12 "HPD" I L 7050 1950 50
 F13 "HDMI_5V" I L 7050 2100 50
+F14 "SH" I R 7650 850 50
 $EndSheet
 $Sheet
@@
 F12 "HPD" I L 5250 1950 50
 F13 "HDMI_5V" I L 5250 2100 50
+F14 "SH" I R 5850 850 50
 $EndSheet
 Text Label 4750 2100 0    50   ~ 0
@@
 Entry Wire Line
 	4750 850  4650 950
-$Sheet
-S 5250 2600 600  1600
-U 5F1D1914
-F0 "HDMI_Connector5F1D1913" 50
-F1 "HDMI_Connector.sch" 50
-F2 "D2+" I L 5250 2800 50
-F3 "D2-" I L 5250 2900 50
-F4 "D1+" I L 5250 3000 50
-F5 "D1-" I L 5250 3100 50
-F6 "D0+" I L 5250 3200 50
-F7 "D0-" I L 5250 3300 50
-F8 "CK+" I L 5250 3400 50
-F9 "CK-" I L 5250 3500 50
-F10 "SCL" I L 5250 3650 50
-F11 "SDA" I L 5250 3750 50
-F12 "HPD" I L 5250 3900 50
-F13 "HDMI_5V" I L 5250 4050 50
-$EndSheet
 Wire Wire Line
 	9950 3950 9200 3950
@@
 F12 "HPD" I L 9950 5050 50
 F13 "HDMI_5V" I L 9950 5200 50
+F14 "SH" I R 10550 3950 50
 $EndSheet
 $Sheet
@@
 F12 "HPD" I L 8100 5100 50
 F13 "HDMI_5V" I L 8100 5250 50
+F14 "SH" I R 8700 4000 50
 $EndSheet
 Entry Wire Line
@@
 	9950 5200 9200 5200
 Wire Notes Line
-	6250 4300 6250 2650
+	6200 4300 6200 2650
 Wire Notes Line
 	9850 2650 9850 500
@@
 	7050 850  6550 850
 Wire Wire Line
-	5250 4050 4750 4050
-Wire Wire Line
-	5250 3900 4750 3900
-Wire Wire Line
-	4750 3750 5250 3750
-Wire Wire Line
-	5250 3650 4750 3650
-Wire Wire Line
-	5250 3500 4750 3500
-Wire Wire Line
-	5250 3400 4750 3400
-Wire Wire Line
-	5250 3300 4750 3300
-Wire Wire Line
-	5250 3200 4750 3200
-Wire Wire Line
-	5250 3100 4750 3100
-Wire Wire Line
-	5250 3000 4750 3000
-Wire Wire Line
-	5250 2900 4750 2900
-Wire Wire Line
-	5250 2800 4750 2800
+	5200 4050 4750 4050
+Wire Wire Line
+	5200 3900 4750 3900
+Wire Wire Line
+	4750 3750 5200 3750
+Wire Wire Line
+	5200 3650 4750 3650
+Wire Wire Line
+	5200 3500 4750 3500
+Wire Wire Line
+	5200 3400 4750 3400
+Wire Wire Line
+	5200 3300 4750 3300
+Wire Wire Line
+	5200 3200 4750 3200
+Wire Wire Line
+	5200 3100 4750 3100
+Wire Wire Line
+	5200 3000 4750 3000
+Wire Wire Line
+	5200 2900 4750 2900
+Wire Wire Line
+	5200 2800 4750 2800
 Wire Wire Line
 	4750 2100 5250 2100
@@
 Text Notes 7150 2500 0    50   ~ 0
 HDMI input
+Text GLabel 6000 1700 3    50   Input ~ 0
+SHIELD
+Text GLabel 8800 4100 3    50   Input ~ 0
+SHIELD
+Text GLabel 10650 4050 3    50   Input ~ 0
+SHIELD
+$Comp
+L Device:R R?
+U 1 1 5F20B45F
+P 6000 1400
+F 0 "R?" H 6070 1446 50  0000 L CNN
+F 1 "R0" H 6070 1355 50  0000 L CNN
+F 2 "" V 5930 1400 50  0001 C CNN
+F 3 "~" H 6000 1400 50  0001 C CNN
+	1    6000 1400
+	1    0    0    -1
+$EndComp
+Wire Wire Line
+	6000 1700 6000 1550
+Wire Wire Line
+	6000 1250 6000 850
+Wire Wire Line
+	5850 850  6000 850
+Text GLabel 7850 1700 3    50   Input ~ 0
+SHIELD
+$Comp
+L Device:R R?
+U 1 1 5F326206
+P 7850 1400
+F 0 "R?" H 7920 1446 50  0000 L CNN
+F 1 "R0" H 7920 1355 50  0000 L CNN
+F 2 "" V 7780 1400 50  0001 C CNN
+F 3 "~" H 7850 1400 50  0001 C CNN
+	1    7850 1400
+	1    0    0    -1
+$EndComp
+Wire Wire Line
+	7850 1700 7850 1550
+Wire Wire Line
+	7850 1250 7850 850
+Wire Wire Line
+	7650 850  7850 850
+Text GLabel 9450 1700 3    50   Input ~ 0
+SHIELD
+$Comp
+L Device:R R?
+U 1 1 5F342D93
+P 9450 1400
+F 0 "R?" H 9520 1446 50  0000 L CNN
+F 1 "R0" H 9520 1355 50  0000 L CNN
+F 2 "" V 9380 1400 50  0001 C CNN
+F 3 "~" H 9450 1400 50  0001 C CNN
+	1    9450 1400
+	1    0    0    -1
+$EndComp
+Wire Wire Line
+	9450 1700 9450 1550
+Wire Wire Line
+	9450 1250 9450 850
+Wire Wire Line
+	9250 850  9450 850
+Text GLabel 6000 3650 3    50   Input ~ 0
+SHIELD
+$Comp
+L Device:R R?
+U 1 1 5F35FBB0
+P 6000 3350
+F 0 "R?" H 6070 3396 50  0000 L CNN
+F 1 "R0" H 6070 3305 50  0000 L CNN
+F 2 "" V 5930 3350 50  0001 C CNN
+F 3 "~" H 6000 3350 50  0001 C CNN
+	1    6000 3350
+	1    0    0    -1
+$EndComp
+$Sheet
+S 5200 2600 600  1600
+U 5F1D1914
+F0 "HDMI_Connector5F1D1913" 50
+F1 "HDMI_Connector.sch" 50
+F2 "D2+" I L 5200 2800 50
+F3 "D2-" I L 5200 2900 50
+F4 "D1+" I L 5200 3000 50
+F5 "D1-" I L 5200 3100 50
+F6 "D0+" I L 5200 3200 50
+F7 "D0-" I L 5200 3300 50
+F8 "CK+" I L 5200 3400 50
+F9 "CK-" I L 5200 3500 50
+F10 "SCL" I L 5200 3650 50
+F11 "SDA" I L 5200 3750 50
+F12 "HPD" I L 5200 3900 50
+F13 "HDMI_5V" I L 5200 4050 50
+F14 "SH" I R 5800 2800 50
+$EndSheet
+Wire Wire Line
+	6000 3650 6000 3500
+Wire Wire Line
+	6000 3200 6000 2800
+Wire Wire Line
+	6000 2800 5800 2800
+Wire Wire Line
+	10550 3950 10650 3950
+Wire Wire Line
+	10650 3950 10650 4050
+Wire Wire Line
+	8700 4000 8800 4000
+Wire Wire Line
+	8800 4000 8800 4100
 Wire Bus Line
 	4650 2750 4650 4250
